File: hardware/pcb/plate_A.kicad_pcb (KiCad board)
At the start: 2 copper layers, 100 x 80 mm, 51 parts, among them J10 OLED GND VDD SCK SDA, J11 BTN, J12 SPI резерв 3V3 GND SCK MISO M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, J3 mACS1 VCC GND VIOUT FAULT, J4 mACS2 VCC GND VIOUT FAULT, J5 mACS3 VCC GND VIOUT FAULT, J6 mSW1 GND ON, J7 mSW2 GND ON, J8 mREL2 GND IN1 IN2 VCC JD-VCC, J9 DPS GND TX RX, Q1 BC547, Q2 BC547, Q3 BC557, X1 B1 B2 GND (L01 L02 P28), X2 VIN_DC GND → mDC5 IN (L03 L04), X3 +5V GND ← mDC5 OUT (L05 L06), X4 DS18B20 ×2: 3V3 DATA GND, X5 U_LOAD_SENSE ← LOAD+ (плата B)

Commit message: Refactor code structure for improved readability and maintainability
Parts:
- R1, R10, R11, R12, R13, R14, R15, R16, R17, R18, R2, R3, R4, R5, R6, R7, R8, R9: footprint R_Axial_DIN0207_L6.3mm_D2.5mm_P10.16mm_Horizontal -> R_1206_3216Metric
- moved Q1 15.4 mm to (59.3, 54.8)
- moved Q2 15.4 mm to (59.3, 61.8)
- moved Q3 15.4 mm to (59.3, 47.8)
- moved C3 15.4 mm to (59.3, 26.5)
- moved C4 15.4 mm to (59.3, 31.5)
- moved C5 15.4 mm to (59.3, 36.5)
- moved C6 15.4 mm to (59.3, 41.5)
- moved C9 15.4 mm to (59.3, 21.5)
- moved VD2 7.70 mm to (61.9, 67.6)
- moved VD1 7.70 mm to (47.5, 67.6)
- moved C7 7.70 mm to (53.2, 16.5)
- moved C8 7.70 mm to (61.8, 16.5)
- moved R11 6.48 mm to (54.4, 41.2)
- moved R13 6.48 mm to (54.4, 46.2)
- moved R15 6.48 mm to (54.4, 53.2)
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