File: hardware/schematic/logic.kicad_sch (KiCad schematic)
At the start: 28 parts, among them J10 OLED GND VDD SCK SDA, J11 BTN, J12 SPI резерв 3V3 GND SCK MISO M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, J6 mSW1 GND ON, J7 mSW2 GND ON, J8 mREL2 GND IN1 IN2 VCC JD-VCC, J9 DPS GND TX RX, Q1 BC547, Q2 BC547, SW1 кнопка панелі, T1 DS18B20 Bat1, T2 DS18B20 Bat2, X1 B1 B2 GND (L01 L02 P28), X2 VIN_DC GND → mDC5 IN (L03 L04), X3 +5V GND ← mDC5 OUT (L05 L06), X4 DS18B20 ×2: 3V3 DATA GND

Commit message: Refactor code structure for improved readability and maintainability
Parts:
- R12, R13, R14, R15, R16, R17, R18: footprint Resistor_THT:R_Axial_DIN0207_L6.3mm_D2.5mm_P10.16mm_Horizontal -> Resistor_SMD:R_1206_3216Metric
Changed lines of the file:
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@@
     (instances
       (project "batman"
-        (path "/bb117f8f-5cc8-4cab-befe-830f3e1e9ea9/4b1c012a-fc93-4450-8aad-b013cfa30a54"
+        (path "/5fff83d6-d1f8-41ff-8dda-774162ba8761/0d95c7f9-4f22-41d9-9831-fe7d3f3e3821"
           (reference "mMCU")
           (unit 1)
@@
     (instances
       (project "batman"
-        (path "/bb117f8f-5cc8-4cab-befe-830f3e1e9ea9/4b1c012a-fc93-4450-8aad-b013cfa30a54"
+        (path "/5fff83d6-d1f8-41ff-8dda-774162ba8761/0d95c7f9-4f22-41d9-9831-fe7d3f3e3821"
           (reference "Q1")
           (unit 1)
@@
       )
     )
-    (property "Footprint" "Resistor_THT:R_Axial_DIN0207_L6.3mm_D2.5mm_P10.16mm_Horizontal"
+    (property "Footprint" "Resistor_SMD:R_1206_3216Metric"
       (at 160.02 59.69 0)
       (effects
@@
     (instances
       (project "batman"
-        (path "/bb117f8f-5cc8-4cab-befe-830f3e1e9ea9/4b1c012a-fc93-4450-8aad-b013cfa30a54"
+        (path "/5fff83d6-d1f8-41ff-8dda-774162ba8761/0d95c7f9-4f22-41d9-9831-fe7d3f3e3821"
           (reference "R12")
           (unit 1)
@@
       )
     )
-    (property "Footprint" "Resistor_THT:R_Axial_DIN0207_L6.3mm_D2.5mm_P10.16mm_Horizontal"
+    (property "Footprint" "Resistor_SMD:R_1206_3216Metric"
       (at 190.5 90.17 0)
       (effects
@@
     (instances
       (project "batman"
-        (path "/bb117f8f-5cc8-4cab-befe-830f3e1e9ea9/4b1c012a-fc93-4450-8aad-b013cfa30a54"
+        (path "/5fff83d6-d1f8-41ff-8dda-774162ba8761/0d95c7f9-4f22-41d9-9831-fe7d3f3e3821"
           (reference "R13")
           (unit 1)
@@
     (instances
       (project "batman"
-        (path "/bb117f8f-5cc8-4cab-befe-830f3e1e9ea9/4b1c012a-fc93-4450-8aad-b013cfa30a54"
+        (path "/5fff83d6-d1f8-41ff-8dda-774162ba8761/0d95c7f9-4f22-41d9-9831-fe7d3f3e3821"
           (reference "Q2")
           (unit 1)
@@
       )
     )
-    (property "Footprint" "Resistor_THT:R_Axial_DIN0207_L6.3mm_D2.5mm_P10.16mm_Horizontal"
+    (property "Footprint" "Resistor_SMD:R_1206_3216Metric"
       (at 160.02 129.54 0)
       (effects
@@
     (instances
       (project "batman"
-        (path "/bb117f8f-5cc8-4cab-befe-830f3e1e9ea9/4b1c012a-fc93-4450-8aad-b013cfa30a54"
+        (path "/5fff83d6-d1f8-41ff-8dda-774162ba8761/0d95c7f9-4f22-41d9-9831-fe7d3f3e3821"
           (reference "R14")
           (unit 1)
@@
       )
     )
-    (property "Footprint" "Resistor_THT:R_Axial_DIN0207_L6.3mm_D2.5mm_P10.16mm_Horizontal"
+    (property "Footprint" "Resistor_SMD:R_1206_3216Metric"
       (at 190.5 160.02 0)
       (effects
@@
     (instances
       (project "batman"
-        (path "/bb117f8f-5cc8-4cab-befe-830f3e1e9ea9/4b1c012a-fc93-4450-8aad-b013cfa30a54"
+        (path "/5fff83d6-d1f8-41ff-8dda-774162ba8761/0d95c7f9-4f22-41d9-9831-fe7d3f3e3821"
           (reference "R15")
           (unit 1)
@@
     (instances
       (project "batman"
-        (path "/bb117f8f-5cc8-4cab-befe-830f3e1e9ea9/4b1c012a-fc93-4450-8aad-b013cfa30a54"
+        (path "/5fff83d6-d1f8-41ff-8dda-774162ba8761/0d95c7f9-4f22-41d9-9831-fe7d3f3e3821"
           (reference "J8")
           (unit 1)
@@
     (instances
       (project "batman"
-        (path "/bb117f8f-5cc8-4cab-befe-830f3e1e9ea9/4b1c012a-fc93-4450-8aad-b013cfa30a54"
+        (path "/5fff83d6-d1f8-41ff-8dda-774162ba8761/0d95c7f9-4f22-41d9-9831-fe7d3f3e3821"
           (reference "J6")
           (unit 1)
@@
     (instances
       (project "batman"
-        (path "/bb117f8f-5cc8-4cab-befe-830f3e1e9ea9/4b1c012a-fc93-4450-8aad-b013cfa30a54"
+        (path "/5fff83d6-d1f8-41ff-8dda-774162ba8761/0d95c7f9-4f22-41d9-9831-fe7d3f3e3821"
           (reference "J7")
           (unit 1)
@@
     (instances
       (project "batman"
-        (path "/bb117f8f-5cc8-4cab-befe-830f3e1e9ea9/4b1c012a-fc93-4450-8aad-b013cfa30a54"
+        (path "/5fff83d6-d1f8-41ff-8dda-774162ba8761/0d95c7f9-4f22-41d9-9831-fe7d3f3e3821"
           (reference "J9")
           (unit 1)
@@
     (instances
       (project "batman"
-        (path "/bb117f8f-5cc8-4cab-befe-830f3e1e9ea9/4b1c012a-fc93-4450-8aad-b013cfa30a54"
+        (path "/5fff83d6-d1f8-41ff-8dda-774162ba8761/0d95c7f9-4f22-41d9-9831-fe7d3f3e3821"
           (reference "J10")
           (unit 1)
@@
     (instances
       (project "batman"
-        (path "/bb117f8f-5cc8-4cab-befe-830f3e1e9ea9/4b1c012a-fc93-4450-8aad-b013cfa30a54"
+        (path "/5fff83d6-d1f8-41ff-8dda-774162ba8761/0d95c7f9-4f22-41d9-9831-fe7d3f3e3821"
           (reference "mOLED")
           (unit 1)
@@
     (instances
       (project "batman"
-        (path "/bb117f8f-5cc8-4cab-befe-830f3e1e9ea9/4b1c012a-fc93-4450-8aad-b013cfa30a54"
+        (path "/5fff83d6-d1f8-41ff-8dda-774162ba8761/0d95c7f9-4f22-41d9-9831-fe7d3f3e3821"
           (reference "J11")
           (unit 1)
@@
     (instances
       (project "batman"
-        (path "/bb117f8f-5cc8-4cab-befe-830f3e1e9ea9/4b1c012a-fc93-4450-8aad-b013cfa30a54"
+        (path "/5fff83d6-d1f8-41ff-8dda-774162ba8761/0d95c7f9-4f22-41d9-9831-fe7d3f3e3821"
           (reference "SW1")
           (unit 1)
@@
     (instances
       (project "batman"
-        (path "/bb117f8f-5cc8-4cab-befe-830f3e1e9ea9/4b1c012a-fc93-4450-8aad-b013cfa30a54"
+        (path "/5fff83d6-d1f8-41ff-8dda-774162ba8761/0d95c7f9-4f22-41d9-9831-fe7d3f3e3821"
           (reference "J12")
           (unit 1)
@@
       )
     )
-    (property "Footprint" "Resistor_THT:R_Axial_DIN0207_L6.3mm_D2.5mm_P10.16mm_Horizontal"
+    (property "Footprint" "Resistor_SMD:R_1206_3216Metric"
       (at 160.02 199.39 0)
       (effects
@@
     (instances
       (project "batman"
-        (path "/bb117f8f-5cc8-4cab-befe-830f3e1e9ea9/4b1c012a-fc93-4450-8aad-b013cfa30a54"
+        (path "/5fff83d6-d1f8-41ff-8dda-774162ba8761/0d95c7f9-4f22-41d9-9831-fe7d3f3e3821"
           (reference "R16")
           (unit 1)
@@
       )
     )
-    (property "Footprint" "Resistor_THT:R_Axial_DIN0207_L6.3mm_D2.5mm_P10.16mm_Horizontal"
+    (property "Footprint" "Resistor_SMD:R_1206_3216Metric"
       (at 175.26 199.39 0)
       (effects
@@
     (instances
       (project "batman"
-        (path "/bb117f8f-5cc8-4cab-befe-830f3e1e9ea9/4b1c012a-fc93-4450-8aad-b013cfa30a54"
+        (path "/5fff83d6-d1f8-41ff-8dda-774162ba8761/0d95c7f9-4f22-41d9-9831-fe7d3f3e3821"
           (reference "R17")
           (unit 1)
@@
       )
     )
-    (property "Footprint" "Resistor_THT:R_Axial_DIN0207_L6.3mm_D2.5mm_P10.16mm_Horizontal"
+    (property "Footprint" "Resistor_SMD:R_1206_3216Metric"
       (at 190.5 199.39 0)
       (effects
@@
     (instances
       (project "batman"
-        (path "/bb117f8f-5cc8-4cab-befe-830f3e1e9ea9/4b1c012a-fc93-4450-8aad-b013cfa30a54"
+        (path "/5fff83d6-d1f8-41ff-8dda-774162ba8761/0d95c7f9-4f22-41d9-9831-fe7d3f3e3821"
           (reference "R18")
           (unit 1)
@@
     (instances
       (project "batman"
-        (path "/bb117f8f-5cc8-4cab-befe-830f3e1e9ea9/4b1c012a-fc93-4450-8aad-b013cfa30a54"
+        (path "/5fff83d6-d1f8-41ff-8dda-774162ba8761/0d95c7f9-4f22-41d9-9831-fe7d3f3e3821"
           (reference "X1")
           (unit 1)
@@
     (instances
       (project "batman"
-        (path "/bb117f8f-5cc8-4cab-befe-830f3e1e9ea9/4b1c012a-fc93-4450-8aad-b013cfa30a54"
+        (path "/5fff83d6-d1f8-41ff-8dda-774162ba8761/0d95c7f9-4f22-41d9-9831-fe7d3f3e3821"
           (reference "VD1")
           (unit 1)
@@
     (instances
       (project "batman"
-        (path "/bb117f8f-5cc8-4cab-befe-830f3e1e9ea9/4b1c012a-fc93-4450-8aad-b013cfa30a54"
+        (path "/5fff83d6-d1f8-41ff-8dda-774162ba8761/0d95c7f9-4f22-41d9-9831-fe7d3f3e3821"
           (reference "VD2")
           (unit 1)
@@
     (instances
       (project "batman"
-        (path "/bb117f8f-5cc8-4cab-befe-830f3e1e9ea9/4b1c012a-fc93-4450-8aad-b013cfa30a54"
+        (path "/5fff83d6-d1f8-41ff-8dda-774162ba8761/0d95c7f9-4f22-41d9-9831-fe7d3f3e3821"
           (reference "X2")
           (unit 1)
@@
     (instances
       (project "batman"
-        (path "/bb117f8f-5cc8-4cab-befe-830f3e1e9ea9/4b1c012a-fc93-4450-8aad-b013cfa30a54"
+        (path "/5fff83d6-d1f8-41ff-8dda-774162ba8761/0d95c7f9-4f22-41d9-9831-fe7d3f3e3821"
           (reference "mDC5")
           (unit 1)
@@
     (instances
       (project "batman"
-        (path "/bb117f8f-5cc8-4cab-befe-830f3e1e9ea9/4b1c012a-fc93-4450-8aad-b013cfa30a54"
+        (path "/5fff83d6-d1f8-41ff-8dda-774162ba8761/0d95c7f9-4f22-41d9-9831-fe7d3f3e3821"
           (reference "X3")
           (unit 1)
@@
     (instances
       (project "batman"
-        (path "/bb117f8f-5cc8-4cab-befe-830f3e1e9ea9/4b1c012a-fc93-4450-8aad-b013cfa30a54"
+        (path "/5fff83d6-d1f8-41ff-8dda-774162ba8761/0d95c7f9-4f22-41d9-9831-fe7d3f3e3821"
           (reference "#FLG6")
           (unit 1)
@@
     (instances
       (project "batman"
-        (path "/bb117f8f-5cc8-4cab-befe-830f3e1e9ea9/4b1c012a-fc93-4450-8aad-b013cfa30a54"
+        (path "/5fff83d6-d1f8-41ff-8dda-774162ba8761/0d95c7f9-4f22-41d9-9831-fe7d3f3e3821"
           (reference "X4")
           (unit 1)
@@
     (instances
       (project "batman"
-        (path "/bb117f8f-5cc8-4cab-befe-830f3e1e9ea9/4b1c012a-fc93-4450-8aad-b013cfa30a54"
+        (path "/5fff83d6-d1f8-41ff-8dda-774162ba8761/0d95c7f9-4f22-41d9-9831-fe7d3f3e3821"
           (reference "T1")
           (unit 1)
@@
     (instances
       (project "batman"
-        (path "/bb117f8f-5cc8-4cab-befe-830f3e1e9ea9/4b1c012a-fc93-4450-8aad-b013cfa30a54"
+        (path "/5fff83d6-d1f8-41ff-8dda-774162ba8761/0d95c7f9-4f22-41d9-9831-fe7d3f3e3821"
           (reference "T2")
           (unit 1)
