File: hardware/schematic/sense.kicad_sch (KiCad schematic)
At the start: 24 parts, among them J3 mACS1 VCC GND VIOUT FAULT, J4 mACS2 VCC GND VIOUT FAULT, J5 mACS3 VCC GND VIOUT FAULT, Q3 BC557, X5 U_LOAD_SENSE ← LOAD+ (плата B)

Commit message: Refactor code structure for improved readability and maintainability
Parts:
- R1, R10, R11, R2, R3, R4, R5, R6, R7, R8, R9: footprint Resistor_THT:R_Axial_DIN0207_L6.3mm_D2.5mm_P10.16mm_Horizontal -> Resistor_SMD:R_1206_3216Metric
Changed lines of the file:
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@@
     (instances
       (project "batman"
-        (path "/bb117f8f-5cc8-4cab-befe-830f3e1e9ea9/f6521d3a-7bbc-4cb4-b5e1-44cfdd4ad4aa"
+        (path "/5fff83d6-d1f8-41ff-8dda-774162ba8761/650ac2d8-5daf-4e26-b148-75134734ae5f"
           (reference "J3")
           (unit 1)
@@
     (instances
       (project "batman"
-        (path "/bb117f8f-5cc8-4cab-befe-830f3e1e9ea9/f6521d3a-7bbc-4cb4-b5e1-44cfdd4ad4aa"
+        (path "/5fff83d6-d1f8-41ff-8dda-774162ba8761/650ac2d8-5daf-4e26-b148-75134734ae5f"
           (reference "J4")
           (unit 1)
@@
     (instances
       (project "batman"
-        (path "/bb117f8f-5cc8-4cab-befe-830f3e1e9ea9/f6521d3a-7bbc-4cb4-b5e1-44cfdd4ad4aa"
+        (path "/5fff83d6-d1f8-41ff-8dda-774162ba8761/650ac2d8-5daf-4e26-b148-75134734ae5f"
           (reference "J5")
           (unit 1)
@@
       )
     )
-    (property "Footprint" "Resistor_THT:R_Axial_DIN0207_L6.3mm_D2.5mm_P10.16mm_Horizontal"
+    (property "Footprint" "Resistor_SMD:R_1206_3216Metric"
       (at 90.17 59.69 0)
       (effects
@@
     (instances
       (project "batman"
-        (path "/bb117f8f-5cc8-4cab-befe-830f3e1e9ea9/f6521d3a-7bbc-4cb4-b5e1-44cfdd4ad4aa"
+        (path "/5fff83d6-d1f8-41ff-8dda-774162ba8761/650ac2d8-5daf-4e26-b148-75134734ae5f"
           (reference "R7")
           (unit 1)
@@
     (instances
       (project "batman"
-        (path "/bb117f8f-5cc8-4cab-befe-830f3e1e9ea9/f6521d3a-7bbc-4cb4-b5e1-44cfdd4ad4aa"
+        (path "/5fff83d6-d1f8-41ff-8dda-774162ba8761/650ac2d8-5daf-4e26-b148-75134734ae5f"
           (reference "C7")
           (unit 1)
@@
       )
     )
-    (property "Footprint" "Resistor_THT:R_Axial_DIN0207_L6.3mm_D2.5mm_P10.16mm_Horizontal"
+    (property "Footprint" "Resistor_SMD:R_1206_3216Metric"
       (at 90.17 100.33 0)
       (effects
@@
     (instances
       (project "batman"
-        (path "/bb117f8f-5cc8-4cab-befe-830f3e1e9ea9/f6521d3a-7bbc-4cb4-b5e1-44cfdd4ad4aa"
+        (path "/5fff83d6-d1f8-41ff-8dda-774162ba8761/650ac2d8-5daf-4e26-b148-75134734ae5f"
           (reference "R8")
           (unit 1)
@@
     (instances
       (project "batman"
-        (path "/bb117f8f-5cc8-4cab-befe-830f3e1e9ea9/f6521d3a-7bbc-4cb4-b5e1-44cfdd4ad4aa"
+        (path "/5fff83d6-d1f8-41ff-8dda-774162ba8761/650ac2d8-5daf-4e26-b148-75134734ae5f"
           (reference "C8")
           (unit 1)
@@
       )
     )
-    (property "Footprint" "Resistor_THT:R_Axial_DIN0207_L6.3mm_D2.5mm_P10.16mm_Horizontal"
+    (property "Footprint" "Resistor_SMD:R_1206_3216Metric"
       (at 90.17 139.7 0)
       (effects
@@
     (instances
       (project "batman"
-        (path "/bb117f8f-5cc8-4cab-befe-830f3e1e9ea9/f6521d3a-7bbc-4cb4-b5e1-44cfdd4ad4aa"
+        (path "/5fff83d6-d1f8-41ff-8dda-774162ba8761/650ac2d8-5daf-4e26-b148-75134734ae5f"
           (reference "R9")
           (unit 1)
@@
     (instances
       (project "batman"
-        (path "/bb117f8f-5cc8-4cab-befe-830f3e1e9ea9/f6521d3a-7bbc-4cb4-b5e1-44cfdd4ad4aa"
+        (path "/5fff83d6-d1f8-41ff-8dda-774162ba8761/650ac2d8-5daf-4e26-b148-75134734ae5f"
           (reference "C9")
           (unit 1)
@@
       )
     )
-    (property "Footprint" "Resistor_THT:R_Axial_DIN0207_L6.3mm_D2.5mm_P10.16mm_Horizontal"
+    (property "Footprint" "Resistor_SMD:R_1206_3216Metric"
       (at 90.17 190.5 0)
       (effects
@@
     (instances
       (project "batman"
-        (path "/bb117f8f-5cc8-4cab-befe-830f3e1e9ea9/f6521d3a-7bbc-4cb4-b5e1-44cfdd4ad4aa"
+        (path "/5fff83d6-d1f8-41ff-8dda-774162ba8761/650ac2d8-5daf-4e26-b148-75134734ae5f"
           (reference "R1")
           (unit 1)
@@
       )
     )
-    (property "Footprint" "Resistor_THT:R_Axial_DIN0207_L6.3mm_D2.5mm_P10.16mm_Horizontal"
+    (property "Footprint" "Resistor_SMD:R_1206_3216Metric"
       (at 119.38 190.5 0)
       (effects
@@
     (instances
       (project "batman"
-        (path "/bb117f8f-5cc8-4cab-befe-830f3e1e9ea9/f6521d3a-7bbc-4cb4-b5e1-44cfdd4ad4aa"
+        (path "/5fff83d6-d1f8-41ff-8dda-774162ba8761/650ac2d8-5daf-4e26-b148-75134734ae5f"
           (reference "R2")
           (unit 1)
@@
     (instances
       (project "batman"
-        (path "/bb117f8f-5cc8-4cab-befe-830f3e1e9ea9/f6521d3a-7bbc-4cb4-b5e1-44cfdd4ad4aa"
+        (path "/5fff83d6-d1f8-41ff-8dda-774162ba8761/650ac2d8-5daf-4e26-b148-75134734ae5f"
           (reference "C3")
           (unit 1)
@@
       )
     )
-    (property "Footprint" "Resistor_THT:R_Axial_DIN0207_L6.3mm_D2.5mm_P10.16mm_Horizontal"
+    (property "Footprint" "Resistor_SMD:R_1206_3216Metric"
       (at 90.17 229.87 0)
       (effects
@@
     (instances
       (project "batman"
-        (path "/bb117f8f-5cc8-4cab-befe-830f3e1e9ea9/f6521d3a-7bbc-4cb4-b5e1-44cfdd4ad4aa"
+        (path "/5fff83d6-d1f8-41ff-8dda-774162ba8761/650ac2d8-5daf-4e26-b148-75134734ae5f"
           (reference "R3")
           (unit 1)
@@
       )
     )
-    (property "Footprint" "Resistor_THT:R_Axial_DIN0207_L6.3mm_D2.5mm_P10.16mm_Horizontal"
+    (property "Footprint" "Resistor_SMD:R_1206_3216Metric"
       (at 119.38 229.87 0)
       (effects
@@
     (instances
       (project "batman"
-        (path "/bb117f8f-5cc8-4cab-befe-830f3e1e9ea9/f6521d3a-7bbc-4cb4-b5e1-44cfdd4ad4aa"
+        (path "/5fff83d6-d1f8-41ff-8dda-774162ba8761/650ac2d8-5daf-4e26-b148-75134734ae5f"
           (reference "R4")
           (unit 1)
@@
     (instances
       (project "batman"
-        (path "/bb117f8f-5cc8-4cab-befe-830f3e1e9ea9/f6521d3a-7bbc-4cb4-b5e1-44cfdd4ad4aa"
+        (path "/5fff83d6-d1f8-41ff-8dda-774162ba8761/650ac2d8-5daf-4e26-b148-75134734ae5f"
           (reference "C4")
           (unit 1)
@@
       )
     )
-    (property "Footprint" "Resistor_THT:R_Axial_DIN0207_L6.3mm_D2.5mm_P10.16mm_Horizontal"
+    (property "Footprint" "Resistor_SMD:R_1206_3216Metric"
       (at 90.17 270.51 0)
       (effects
@@
     (instances
       (project "batman"
-        (path "/bb117f8f-5cc8-4cab-befe-830f3e1e9ea9/f6521d3a-7bbc-4cb4-b5e1-44cfdd4ad4aa"
+        (path "/5fff83d6-d1f8-41ff-8dda-774162ba8761/650ac2d8-5daf-4e26-b148-75134734ae5f"
           (reference "R5")
           (unit 1)
@@
       )
     )
-    (property "Footprint" "Resistor_THT:R_Axial_DIN0207_L6.3mm_D2.5mm_P10.16mm_Horizontal"
+    (property "Footprint" "Resistor_SMD:R_1206_3216Metric"
       (at 119.38 270.51 0)
       (effects
@@
     (instances
       (project "batman"
-        (path "/bb117f8f-5cc8-4cab-befe-830f3e1e9ea9/f6521d3a-7bbc-4cb4-b5e1-44cfdd4ad4aa"
+        (path "/5fff83d6-d1f8-41ff-8dda-774162ba8761/650ac2d8-5daf-4e26-b148-75134734ae5f"
           (reference "R6")
           (unit 1)
@@
     (instances
       (project "batman"
-        (path "/bb117f8f-5cc8-4cab-befe-830f3e1e9ea9/f6521d3a-7bbc-4cb4-b5e1-44cfdd4ad4aa"
+        (path "/5fff83d6-d1f8-41ff-8dda-774162ba8761/650ac2d8-5daf-4e26-b148-75134734ae5f"
           (reference "C5")
           (unit 1)
@@
     (instances
       (project "batman"
-        (path "/bb117f8f-5cc8-4cab-befe-830f3e1e9ea9/f6521d3a-7bbc-4cb4-b5e1-44cfdd4ad4aa"
+        (path "/5fff83d6-d1f8-41ff-8dda-774162ba8761/650ac2d8-5daf-4e26-b148-75134734ae5f"
           (reference "X5")
           (unit 1)
@@
     (instances
       (project "batman"
-        (path "/bb117f8f-5cc8-4cab-befe-830f3e1e9ea9/f6521d3a-7bbc-4cb4-b5e1-44cfdd4ad4aa"
+        (path "/5fff83d6-d1f8-41ff-8dda-774162ba8761/650ac2d8-5daf-4e26-b148-75134734ae5f"
           (reference "mADC")
           (unit 1)
@@
     (instances
       (project "batman"
-        (path "/bb117f8f-5cc8-4cab-befe-830f3e1e9ea9/f6521d3a-7bbc-4cb4-b5e1-44cfdd4ad4aa"
+        (path "/5fff83d6-d1f8-41ff-8dda-774162ba8761/650ac2d8-5daf-4e26-b148-75134734ae5f"
           (reference "C6")
           (unit 1)
@@
     (instances
       (project "batman"
-        (path "/bb117f8f-5cc8-4cab-befe-830f3e1e9ea9/f6521d3a-7bbc-4cb4-b5e1-44cfdd4ad4aa"
+        (path "/5fff83d6-d1f8-41ff-8dda-774162ba8761/650ac2d8-5daf-4e26-b148-75134734ae5f"
           (reference "Q3")
           (unit 1)
@@
       )
     )
-    (property "Footprint" "Resistor_THT:R_Axial_DIN0207_L6.3mm_D2.5mm_P10.16mm_Horizontal"
+    (property "Footprint" "Resistor_SMD:R_1206_3216Metric"
       (at 279.4 90.17 0)
       (effects
@@
     (instances
       (project "batman"
-        (path "/bb117f8f-5cc8-4cab-befe-830f3e1e9ea9/f6521d3a-7bbc-4cb4-b5e1-44cfdd4ad4aa"
+        (path "/5fff83d6-d1f8-41ff-8dda-774162ba8761/650ac2d8-5daf-4e26-b148-75134734ae5f"
           (reference "R10")
           (unit 1)
@@
       )
     )
-    (property "Footprint" "Resistor_THT:R_Axial_DIN0207_L6.3mm_D2.5mm_P10.16mm_Horizontal"
+    (property "Footprint" "Resistor_SMD:R_1206_3216Metric"
       (at 320.04 49.53 0)
       (effects
@@
     (instances
       (project "batman"
-        (path "/bb117f8f-5cc8-4cab-befe-830f3e1e9ea9/f6521d3a-7bbc-4cb4-b5e1-44cfdd4ad4aa"
+        (path "/5fff83d6-d1f8-41ff-8dda-774162ba8761/650ac2d8-5daf-4e26-b148-75134734ae5f"
           (reference "R11")
           (unit 1)
@@
     (instances
       (project "batman"
-        (path "/bb117f8f-5cc8-4cab-befe-830f3e1e9ea9/f6521d3a-7bbc-4cb4-b5e1-44cfdd4ad4aa"
+        (path "/5fff83d6-d1f8-41ff-8dda-774162ba8761/650ac2d8-5daf-4e26-b148-75134734ae5f"
           (reference "#FLG5")
           (unit 1)
